Commit message: added in measurements of rockie

File: rockie_workspace/src/rockie_core/rockie.urdf (robot description, URDF)
Before this commit: robot rockie, 5 links, 4 joints
Joints:
- removed joint base_link_to_arm_revolute
- added joint corner_to_arm_revolute: type revolute, parent corner, child arm_revolute, origin xyz=0.942975 0.098425 0.73025, axis 0 0 1, limit lower=0 upper=3.14159 effort=1.0 velocity=1.0
- joint arm_prismatic_to_gripper: origin xyz=0 0 -0.5 -> xyz=0 0.053974999999999995 -0.8191499999999999
- joint arm_revolute_to_arm_prismatic: limit lower=0 upper=0.5 effort=1.0 velocity=1.0 -> lower=0 upper=0.542925 effort=1.0 velocity=1.0; origin xyz=0.2 0 0 -> xyz=0.3302 0 0
- joint corner_to_base_link: origin xyz=0.5 0.2 0 -> xyz=0.4572 0.3048 0
