Commit message: network cameras extrinsics calibrated to stereo camera

File: rockie_workspace/src/rockie_core/config/rockie.urdf (robot description, URDF)
Before this commit: robot rockie, 5 links, 4 joints
Links:
- added link /left_camera
- added link /right_camera
- added link stereo_camera
Joints:
- added joint /left_camera_joint: type fixed, parent stereo_camera, child /left_camera, origin xyz=-0.137257 0.105664 0.019686 rpy=0.463344 -0.886846 -0.408139
- added joint /right_camera_joint: type fixed, parent stereo_camera, child /right_camera, origin xyz=0.691138 0.146036 0.124159 rpy=0.132469 0.214288 0.101302
- added joint corner_to_stereo_camera: type fixed, parent corner, child stereo_camera, origin xyz=0.6 0.3 0.5

Commit message: full kinematic calibration of robot and added option for disembodied mode to slam

File: rockie_workspace/src/rockie_core/config/rockie.urdf (robot description, URDF)
Before this commit: robot rockie, 8 links, 7 joints
Links:
- added link stereo_camera_platform
Joints:
- removed joint corner_to_stereo_camera
- added joint corner_to_stereo_camera_platform: type fixed, parent corner, child stereo_camera_platform, origin xyz=0.9017 0 0.6985 rpy=0.0 0.5235987755982988 0.0
- added joint stereo_camera_platform_to_stereo_camera: type fixed, parent stereo_camera_platform, child stereo_camera, origin xyz=0.0333375 0.5651499999999999 0.038099999999999995 rpy=-1.5707963267948966 0 -1.5707963267948966

Commit message: updated camera calibration

File: rockie_workspace/src/rockie_core/config/rockie.urdf (robot description, URDF)
Before this commit: robot rockie, 9 links, 8 joints
Joints:
- joint /left_camera_joint: origin xyz=-0.137257 0.105664 0.019686 rpy=0.463344 -0.886846 -0.408139 -> xyz=-0.163691 0.12499 -0.00243303 rpy=-0.105078 -0.818555 -0.100929
- joint /right_camera_joint: origin xyz=0.691138 0.146036 0.124159 rpy=0.132469 0.214288 0.101302 -> xyz=0.714194 0.0981112 0.0825147 rpy=-0.279391 0.381873 -0.0456388
- joint corner_to_stereo_camera_platform: origin xyz=0.9017 0 0.6985 rpy=0.0 0.5235987755982988 0.0 -> xyz=0.9017 0 0.6985 rpy=0.0 0.2205 0.0

Commit message: making base_link top of root because rtabmap was whining

File: rockie_workspace/src/rockie_core/config/rockie.urdf (robot description, URDF)
Before this commit: robot rockie, 9 links, 8 joints
Joints:
- joint corner_to_base_link: child base_link -> corner; origin xyz=0.4572 0.3048 0 -> xyz=-0.4572 -0.3048 0; parent corner -> base_link

Commit message: wip updates to launch files and current calibration file

File: rockie_workspace/src/rockie_core/config/rockie.urdf (robot description, URDF)
Before this commit: robot rockie, 9 links, 8 joints
Joints:
- joint /left_camera_joint: origin xyz=-0.163691 0.12499 -0.00243303 rpy=-0.105078 -0.818555 -0.100929 -> xyz=0.438921 0.388299 0.553465 rpy=-1.97047 0.0736801 -0.602207; parent stereo_camera -> base_link
- joint /right_camera_joint: origin xyz=0.714194 0.0981112 0.0825147 rpy=-0.279391 0.381873 -0.0456388 -> xyz=0.503612 -0.431403 0.582553 rpy=-1.98201 -0.0148254 -1.97746; parent stereo_camera -> base_link
- joint corner_to_stereo_camera_platform: origin xyz=0.9017 0 0.6985 rpy=0.0 0.2205 0.0 -> xyz=0.9017 0 0.6985 rpy=0.0 0.205949 0.0

Commit message: calibration

File: rockie_workspace/src/rockie_core/config/rockie.urdf (robot description, URDF)
Before this commit: robot rockie, 9 links, 8 joints
Joints:
- joint /left_camera_joint: origin xyz=0.438921 0.388299 0.553465 rpy=-1.97047 0.0736801 -0.602207 -> xyz=0.497246 0.414693 0.599057 rpy=-1.99231 0.0288284 -1.23172
- joint /right_camera_joint: origin xyz=0.503612 -0.431403 0.582553 rpy=-1.98201 -0.0148254 -1.97746 -> xyz=0.424668 -0.614335 0.586433 rpy=-1.92163 -0.0719595 -1.82614
- joint corner_to_stereo_camera_platform: origin xyz=0.9017 0 0.6985 rpy=0.0 0.205949 0.0 -> xyz=0.9017 0 0.6985 rpy=0.0 0.523599 0.0
